File: hardware/kicad/InternetRadioMinibox/InternetRadioMiniBox.sch (KiCad schematic (older format))
At the start: 41 parts, among them IC1 ESP8266, IC2 ATMEGA328P-P, IC3 23K256, J1 Screw_Terminal_1x03, Y1 12 MHz

Commit message: Added slider switch for band selection.
Parts:
- added R?: 10K, symbol R
- added S-BAND: SLIDER_SWITCH_ON-ON, symbol SLIDER_SWITCH_ON-ON
Connections:
- net labels added: A0, A4, A5, PD7
- wire segments 139 -> 165
Changed lines of the file:
@@
 EESchema Schematic File Version 2
+LIBS:InternetRadio-rescue
 LIBS:power
 LIBS:device
@@
 	4400 2800 5300 2800
 Wire Wire Line
-	1350 8300 2800 8300
+	1350 8300 2400 8300
+Wire Wire Line
+	2400 8300 2800 8300
 Wire Wire Line
 	3300 8600 3300 8700
@@
 	11650 9450 10950 9450
 Wire Wire Line
-	4400 2400 5900 2400
-Wire Wire Line
-	4500 1450 4500 4500
+	4400 2400 4500 2400
+Wire Wire Line
+	4500 2400 5900 2400
+Wire Wire Line
+	4500 1450 4500 2400
+Wire Wire Line
+	4500 2400 4500 4500
 Wire Wire Line
 	4500 4500 3500 4500
@@
 	3500 5100 3500 5350
 Wire Wire Line
-	2350 1450 2350 4850
+	2350 1450 2350 2600
+Wire Wire Line
+	2350 2600 2350 4850
 Wire Wire Line
 	3000 2600 2350 2600
@@
 	10200 2200 12350 2200
 Wire Wire Line
-	12350 2200 12350 2450
+	12350 2200 12350 2400
+Wire Wire Line
+	12350 2400 12350 2450
 Wire Wire Line
 	12350 2400 12200 2400
@@
 	11700 2400 11900 2400
 Wire Wire Line
-	11700 2300 11700 2450
+	11700 2300 11700 2400
+Wire Wire Line
+	11700 2400 11700 2450
 Connection ~ 11700 2400
 Connection ~ 12350 2400
@@
 	12350 2750 12350 2750
 Wire Wire Line
-	7600 950  7600 2550
+	7600 950  7600 1100
+Wire Wire Line
+	7600 1100 7600 1600
+Wire Wire Line
+	7600 1600 7600 2550
 Wire Wire Line
 	8300 3900 7600 3900
 Wire Wire Line
-	7600 2850 7600 4100
+	7600 2850 7600 3900
+Wire Wire Line
+	7600 3900 7600 4100
 Connection ~ 7600 3900
 Wire Wire Line
 	8300 3800 8050 3800
 Wire Wire Line
-	8050 2850 8050 4100
-Wire Wire Line
-	8050 1100 8050 2550
+	8050 2850 8050 3800
+Wire Wire Line
+	8050 3800 8050 4100
+Wire Wire Line
+	8050 1100 8050 1900
+Wire Wire Line
+	8050 1900 8050 2550
 Connection ~ 8050 3800
 Wire Wire Line
-	10400 1500 10400 4400
+	10400 1500 10400 3050
+Wire Wire Line
+	10400 3050 10400 4400
 Wire Wire Line
 	10400 3050 10200 3050
@@
 	11250 2950 11250 3400
 Wire Wire Line
-	11250 3400 15300 3400
+	11250 3400 15050 3400
+Wire Wire Line
+	15050 3400 15300 3400
 Wire Wire Line
 	10200 2850 11350 2850
@@
 $EndComp
 Wire Wire Line
-	15050 3400 15050 3650
+	15050 3400 15050 3600
+Wire Wire Line
+	15050 3600 15050 3650
 Connection ~ 15050 3400
 $Comp
@@
 $EndComp
 Wire Wire Line
-	11550 3500 11550 4350
+	11550 3500 11550 3800
+Wire Wire Line
+	11550 3800 11550 4100
+Wire Wire Line
+	11550 4100 11550 4350
 Connection ~ 11550 3800
 Connection ~ 11550 4100
@@
 	11950 9000 12050 9000
 Wire Bus Line
-	1150 6300 14650 6300
+	1150 6300 1250 6300
+Wire Bus Line
+	1250 6300 1400 6300
+Wire Bus Line
+	1400 6300 1550 6300
+Wire Bus Line
+	1550 6300 1700 6300
+Wire Bus Line
+	1700 6300 5200 6300
+Wire Bus Line
+	5200 6300 5400 6300
+Wire Bus Line
+	5400 6300 5600 6300
+Wire Bus Line
+	5600 6300 5800 6300
+Wire Bus Line
+	5800 6300 6000 6300
+Wire Bus Line
+	6000 6300 6200 6300
+Wire Bus Line
+	6200 6300 9850 6300
+Wire Bus Line
+	9850 6300 9950 6300
+Wire Bus Line
+	9950 6300 10050 6300
+Wire Bus Line
+	10050 6300 10150 6300
+Wire Bus Line
+	10150 6300 13100 6300
+Wire Bus Line
+	13100 6300 13300 6300
+Wire Bus Line
+	13300 6300 13500 6300
+Wire Bus Line
+	13500 6300 13700 6300
+Wire Bus Line
+	13700 6300 14650 6300
 Wire Wire Line
 	5100 2900 5100 6200
@@
 Connection ~ 2700 7050
 Wire Wire Line
-	2400 7050 3300 7050
+	2400 7050 2700 7050
+Wire Wire Line
+	2700 7050 3300 7050
 Wire Wire Line
 	2900 1150 2900 1100
 Wire Wire Line
-	2900 1100 4500 1100
+	2900 1100 3700 1100
+Wire Wire Line
+	3700 1100 4500 1100
 Wire Wire Line
 	4500 1100 4500 1150
@@
 	3700 3600 3700 3550
 Wire Wire Line
-	3300 7000 3300 7550
+	3300 7000 3300 7050
+Wire Wire Line
+	3300 7050 3300 7550
 Wire Wire Line
 	8050 1900 8300 1900
 Wire Wire Line
-	7600 1100 10400 1100
+	7600 1100 8050 1100
+Wire Wire Line
+	8050 1100 10400 1100
 Connection ~ 7600 1100
 Connection ~ 8050 1100
 Text Notes 8650 900  0    39   ~ 0
 Replace with ATTINY 84A-SSU (SOIC-14) to save space
+$Comp
+L SLIDER_SWITCH_ON-ON S-BAND
+U 1 1 58C06CE7
+P 15150 5400
+F 0 "S-BAND" H 15150 5150 60  0000 C CNN
+F 1 "SLIDER_SWITCH_ON-ON" H 15150 5250 60  0000 C CNN
+F 2 "" H 15150 5400 60  0001 C CNN
+F 3 "" H 15150 5400 60  0001 C CNN
+	1    15150 5400
+	1    0    0    -1
+$EndComp
+Wire Wire Line
+	14900 5400 14400 5400
+Wire Wire Line
+	14400 5400 14400 5300
+Wire Wire Line
+	15400 5400 15800 5400
+Wire Wire Line
+	15800 5400 15800 5700
+$Comp
+L GND #PWR?
+U 1 1 58C08F09
+P 15800 5700
+F 0 "#PWR?" H 15800 5450 50  0001 C CNN
+F 1 "GND" H 15800 5550 50  0000 C CNN
+F 2 "" H 15800 5700 50  0000 C CNN
+F 3 "" H 15800 5700 50  0000 C CNN
+	1    15800 5700
+	1    0    0    -1
+$EndComp
+$Comp
+L R R?
+U 1 1 58C08FEB
+P 14400 5150
+F 0 "R?" V 14480 5150 50  0000 C CNN
+F 1 "10K" V 14400 5150 50  0000 C CNN
+F 2 "" V 14330 5150 50  0000 C CNN
+F 3 "" H 14400 5150 50  0000 C CNN
+	1    14400 5150
+	1    0    0    -1
+$EndComp
+$Comp
+L +3.3V #PWR?
+U 1 1 58C0AD0F
+P 14400 5000
+F 0 "#PWR?" H 14400 4850 50  0001 C CNN
+F 1 "+3.3V" H 14400 5140 50  0000 C CNN
+F 2 "" H 14400 5000 50  0000 C CNN
+F 3 "" H 14400 5000 50  0000 C CNN
+	1    14400 5000
+	1    0    0    -1
+$EndComp
+Wire Wire Line
+	10200 3900 10200 4100
+Wire Wire Line
+	15150 5350 15150 5100
+Text GLabel 10200 4100 3    60   Input ~ 0
+PD7
+Text GLabel 15150 5100 1    60   Input ~ 0
+PD7
+Text Label 14450 4550 0    60   ~ 0
+A0
+Text Label 14450 3400 0    60   ~ 0
+A5
+Text Label 14450 3200 0    60   ~ 0
+A4
 $EndSCHEMATC

Commit message: Added VS1011, power units and amp
Parts:
- removed AE1: Antenna, symbol Antenna
- removed B1: VS1053_BOARD, symbol VS1053_BOARD
- removed DREQ1, MISO1, MOSI1, SCK1, XCS1, XDCS1, XRST1: EXT-CONN, symbol EXT-CONN
- removed SW_FLASH1, SW_RESET1: SW_PUSH_SMALL_H, symbol SW_PUSH_SMALL_H
- added A1: ANTENNA_RCX, symbol ANTENNA_RCX
- added C10, C11: 1u-100u, symbol CP
- added C12: 250u, symbol CP
- added C13: 50n, symbol C
- added C7, C8: 33p, Capacitors_SMD:C_0805_HandSoldering, symbol C
- added C9: 100n, Capacitors_SMD:C_0805_HandSoldering, symbol C
- added IC4: VS1011e, symbol VS1011e
- added IC5: LM386, Housings_SOIC:SOIC-8-1EP_3.9x4.9mm_Pitch1.27mm, symbol LM386
- added M1, M2, M3: TSR1-2433, maker:TSR1-2433, symbol TSR1-2433
- added R11: 10M, Resistors_SMD:R_0805_HandSoldering, symbol R
- added R12: 100k, Resistors_SMD:R_0805_HandSoldering, symbol R
- added R13, R14, R15, R16: 100K, Resistors_SMD:R_0805_HandSoldering, symbol R
- added R17, R18: 4.7K, symbol R
- added R19: 47K, symbol R
- added R20: 10, symbol R
- added SW1, SW2: SW_PUSH_SMALL, maker:SMALL_PUSH_BUTTON, symbol SW_PUSH_SMALL
- added Y2: 12.228 MHz, symbol Crystal
- C1: renamed from C3; footprint (none) -> Capacitors_SMD:C_0805_HandSoldering
- C2: renamed from C4; footprint (none) -> Capacitors_SMD:C_0805_HandSoldering
- C3: renamed from C1; footprint (none) -> Capacitors_SMD:C_0805_HandSoldering
- C4: renamed from C2; footprint (none) -> Capacitors_SMD:C_0805_HandSoldering
- C5, C6: footprint (none) -> Capacitors_SMD:C_0805_HandSoldering
- IC2: footprint DIL28 -> (none)
- IC3: footprint DIL -> Housings_SOIC:SOIC-8_3.9x4.9mm_Pitch1.27mm
- R1, R10, R2, R3, R4, R9: footprint (none) -> Resistors_SMD:R_0805_HandSoldering
- R5: renamed from R6; footprint (none) -> Resistors_SMD:R_0805_HandSoldering
- R6: renamed from R7; footprint (none) -> Resistors_SMD:R_0805_HandSoldering
- R7: renamed from R8; footprint (none) -> Resistors_SMD:R_0805_HandSoldering
- R8: renamed from R?; footprint (none) -> Resistors_SMD:R_0805_HandSoldering
- renumbered S-BAND to S-BAND1
Connections:
- net labels added: +9V, AUDIO-LEFT, AUDIO-RIGHT, AVDD+3.3V, DVDD+3.3V, Speaker+
- net labels removed: +5V
- wire segments 165 -> 210
- no-connect marks 14 -> 16
Other:
- note added: "3"
- note added: "AMP"
- note added: "Depending on load resistance"
- note added: "Power"
- note removed: "2"
- note removed: "EXT. CONNECTION"

Commit message: Added board connectors
Parts:
- removed EC1-DTR1, EC1-RXD1, EC1-TXD1, EC2-DTR1, EC2-RXD1, EC2-TXD1: EXT-CONN, symbol EXT-CONN
- removed J1: Screw_Terminal_1x03, symbol Screw_Terminal_1x03
- added P1, P3: CONN_01X02, Connect:PINHEAD1-2, symbol CONN_01X02
- added P2: CONN_01X03, Connect:PINHEAD1-3, symbol CONN_01X03
- added P4: CONN_FTDI_ESP8266, Connect:PINHEAD1-6, symbol CONN_01X06
- added P5: ISP6PIN, symbol CONN_02X03
- added P6: CONN_FTDI_AVR, symbol CONN_01X06
- IC1: footprint (none) -> maker:ESP8266-IN-CIRCUIT
- IC4: footprint (none) -> Housings_SOIC:SOIC-28W_7.5x17.9mm_Pitch1.27mm
Connections:
- net labels added: CTS-AVR, CTS-ESP, DTR-AVR, DTR-ESP, RST-AVR, RXI-AVR, RXI-ESP, SPEAKER+, TXO-AVR, TXO-ESP
- net labels removed: Speaker+
- wire segments 210 -> 230
- no-connect marks 16 -> 17
Other:
- note added: "Depending on \nload resistance"
- note added: "FTDI for AVR"
- note added: "FTDI\nfor ESP8266"
- note added: "Front Panel Controller"
- note added: "ISP for AVR (Optional)"
- note added: "Main Processor"
- note added: "Preloaded with Arduino Bootloader"
- note added: "To Speaker"
- note removed: "19 Feb 2017"
- note removed: "3"
- note removed: "Depending on load resistance"
- note removed: "Design: Andrew Doble"
- note removed: "FTDI"
- moved on the sheet: C5, C6, C7, C8, M1, M3, R11, Y2

Commit message: Replaced pot with rotary encoder for volume control. Removed band switch. Plus small changes.
Parts:
- removed D3: BLUE, symbol LED
- removed R2, R3: 12K, Resistors_SMD:R_0805_HandSoldering, symbol R
- removed R7: 165, Resistors_SMD:R_0805_HandSoldering, symbol R
- removed R8: 10K, Resistors_SMD:R_0805_HandSoldering, symbol R
- removed RV-VOLUME1: POT, symbol POT
- removed S-BAND1: SLIDER_SWITCH_ON-ON, symbol SLIDER_SWITCH_ON-ON
- added S?: ROTARY-ENCODER, symbol ROTARY-ENCODER
- R17, R18: Tolerance (none) -> 1%
Connections:
- net labels added: PD2, PD4
- net labels removed: A0, PD7
- wire segments 230 -> 217
- no-connect marks 17 -> 18
Other:
- note added: "ESP8266 Board has 12K pullups \non GPIO0 and CHIP-EN"
- note removed: "ESP8266 Breakout Board\nIn-Line"
Changed lines of the file:
@@
 	7250 6300 7350 6400
-$Comp
-L R R3
-U 1 1 57DF3202
-P 4500 1300
-F 0 "R3" V 4580 1300 50  0000 C CNN
-F 1 "12K" V 4500 1300 50  0000 C CNN
-F 2 "Resistors_SMD:R_0805_HandSoldering" V 4430 1300 50  0001 C CNN
-F 3 "" H 4500 1300 50  0000 C CNN
-	1    4500 1300
-	1    0    0    -1
-$EndComp
 $Comp
 L GND #PWR04
@@
 	1    0    0    -1
 $EndComp
-$Comp
-L R R2
-U 1 1 580CCDC1
-P 2900 1300
-F 0 "R2" V 2980 1300 50  0000 C CNN
-F 1 "12K" V 2900 1300 50  0000 C CNN
-F 2 "Resistors_SMD:R_0805_HandSoldering" V 2830 1300 50  0001 C CNN
-F 3 "" H 2900 1300 50  0000 C CNN
-	1    2900 1300
-	1    0    0    -1
-$EndComp
-Text Notes 2750 900  0    60   ~ 0
-ESP8266 Breakout Board\nIn-Line
 Text Notes 11900 10300 0    118  ~ 24
 Internet Radio
@@
 To 0-135pF Rotary \nVariable Capacitor. \nCase connected \nto ground.
 $Comp
-L POT RV-VOLUME1
-U 1 1 58AB265C
-P 15450 4550
-F 0 "RV-VOLUME1" V 15275 4550 50  0000 C CNN
-F 1 "POT" V 15350 4550 50  0000 C CNN
-F 2 "" H 15450 4550 50  0001 C CNN
-F 3 "" H 15450 4550 50  0000 C CNN
-	1    15450 4550
-	-1   0    0    1
-$EndComp
-$Comp
-L +3.3V #PWR012
-U 1 1 58AB289C
-P 15450 4400
-F 0 "#PWR012" H 15450 4250 50  0001 C CNN
-F 1 "+3.3V" H 15450 4540 50  0000 C CNN
-F 2 "" H 15450 4400 50  0000 C CNN
-F 3 "" H 15450 4400 50  0000 C CNN
-	1    15450 4400
-	1    0    0    -1
-$EndComp
-$Comp
 L GND #PWR013
 U 1 1 58AB28EA
-P 15450 4700
-F 0 "#PWR013" H 15450 4450 50  0001 C CNN
-F 1 "GND" H 15450 4550 50  0000 C CNN
-F 2 "" H 15450 4700 50  0000 C CNN
-F 3 "" H 15450 4700 50  0000 C CNN
-	1    15450 4700
-	1    0    0    -1
-$EndComp
-$Comp
-L LED D3
-U 1 1 58AB93DA
-P 11100 4100
-F 0 "D3" H 11100 4200 50  0000 C CNN
-F 1 "BLUE" H 11100 4000 50  0000 C CNN
-F 2 "" H 11100 4100 50  0001 C CNN
-F 3 "" H 11100 4100 50  0000 C CNN
-	1    11100 4100
-	-1   0    0    -1
+P 14150 4850
+F 0 "#PWR013" H 14150 4600 50  0001 C CNN
+F 1 "GND" H 14150 4700 50  0000 C CNN
+F 2 "" H 14150 4850 50  0000 C CNN
+F 3 "" H 14150 4850 50  0000 C CNN
+	1    14150 4850
+	1    0    0    -1
 $EndComp
 $Comp
@@
 $EndComp
 $Comp
-L R R7
-U 1 1 58ABC56C
-P 11400 4100
-F 0 "R7" V 11480 4100 50  0000 C CNN
-F 1 "165" V 11400 4100 50  0000 C CNN
-F 2 "Resistors_SMD:R_0805_HandSoldering" V 11330 4100 50  0001 C CNN
-F 3 "" H 11400 4100 50  0000 C CNN
-	1    11400 4100
-	0    1    1    0
-$EndComp
-$Comp
 L GND #PWR014
 U 1 1 58ABC5CC
-P 11550 4350
-F 0 "#PWR014" H 11550 4100 50  0001 C CNN
-F 1 "GND" H 11550 4200 50  0000 C CNN
-F 2 "" H 11550 4350 50  0000 C CNN
-F 3 "" H 11550 4350 50  0000 C CNN
-	1    11550 4350
+P 11550 4050
+F 0 "#PWR014" H 11550 3800 50  0001 C CNN
+F 1 "GND" H 11550 3900 50  0000 C CNN
+F 2 "" H 11550 4050 50  0000 C CNN
+F 3 "" H 11550 4050 50  0000 C CNN
+	1    11550 4050
 	1    0    0    -1
 $EndComp
@@
 NoConn ~ 10200 2750
 NoConn ~ 8300 2200
-NoConn ~ 10200 3600
-NoConn ~ 10200 3400
 $Comp
 L +3.3V #PWR015
@@
 Text Notes 8650 900  0    39   ~ 0
 Replace with ATTINY 84A-SSU (SOIC-14) to save space
-$Comp
-L SLIDER_SWITCH_ON-ON S-BAND1
-U 1 1 58C06CE7
-P 15150 5400
-F 0 "S-BAND1" H 15150 5150 60  0000 C CNN
-F 1 "SLIDER_SWITCH_ON-ON" H 15150 5250 60  0000 C CNN
-F 2 "" H 15150 5400 60  0001 C CNN
-F 3 "" H 15150 5400 60  0001 C CNN
-	1    15150 5400
-	1    0    0    -1
-$EndComp
-$Comp
-L GND #PWR018
-U 1 1 58C08F09
-P 15800 5700
-F 0 "#PWR018" H 15800 5450 50  0001 C CNN
-F 1 "GND" H 15800 5550 50  0000 C CNN
-F 2 "" H 15800 5700 50  0000 C CNN
-F 3 "" H 15800 5700 50  0000 C CNN
-	1    15800 5700
-	1    0    0    -1
-$EndComp
-$Comp
-L R R8
-U 1 1 58C08FEB
-P 14400 5150
-F 0 "R8" V 14480 5150 50  0000 C CNN
-F 1 "10K" V 14400 5150 50  0000 C CNN
-F 2 "Resistors_SMD:R_0805_HandSoldering" V 14330 5150 50  0001 C CNN
-F 3 "" H 14400 5150 50  0000 C CNN
-	1    14400 5150
-	1    0    0    -1
-$EndComp
-$Comp
-L +3.3V #PWR019
-U 1 1 58C0AD0F
-P 14400 5000
-F 0 "#PWR019" H 14400 4850 50  0001 C CNN
-F 1 "+3.3V" H 14400 5140 50  0000 C CNN
-F 2 "" H 14400 5000 50  0000 C CNN
-F 3 "" H 14400 5000 50  0000 C CNN
-	1    14400 5000
-	1    0    0    -1
-$EndComp
-Text Label 14450 4550 0    60   ~ 0
-A0
 Text Label 14450 3300 0    60   ~ 0
 A5
@@
 F 2 "" V 12780 8100 50  0001 C CNN
 F 3 "" H 12850 8100 50  0000 C CNN
+F 4 "1%" V 12850 8100 60  0001 C CNN "Tolerance"
 	1    12850 8100
 	0    1    1    0
@@
 F 2 "" V 12780 8450 50  0001 C CNN
 F 3 "" H 12850 8450 50  0000 C CNN
+F 4 "1%" V 12850 8450 60  0001 C CNN "Tolerance"
 	1    12850 8450
 	0    -1   -1   0
@@
 	4400 2400 5900 2400
 Wire Wire Line
-	4500 4500 4500 1450
+	4500 4500 4500 2400
 Wire Wire Line
 	3500 4500 4500 4500
@@
 Wire Wire Line
 	2350 5100 2350 5500
-Wire Wire Line
-	3000 2700 2900 2700
-Wire Wire Line
-	2900 2700 2900 1450
-Wire Notes Line
-	2700 700  2700 3900
-Wire Notes Line
-	2700 3900 5000 3900
-Wire Notes Line
-	5000 3900 5000 700
-Wire Notes Line
-	5000 700  2700 700
 Wire Wire Line
 	10200 2200 12350 2200
@@
 Connection ~ 15050 3300
 Wire Wire Line
-	10200 2450 11450 2450
-Wire Wire Line
 	10200 2950 11250 2950
 Wire Wire Line
-	11450 2450 11450 3050
-Wire Wire Line
-	12150 4550 15300 4550
-Wire Wire Line
-	10200 3800 10850 3800
-Wire Wire Line
-	10850 4100 10950 4100
-Wire Wire Line
 	10200 3700 10950 3700
 Wire Wire Line
@@
 	10200 3500 10950 3500
 Wire Wire Line
-	11550 3500 11550 4350
+	11550 3500 11550 4100
 Connection ~ 11550 3800
-Connection ~ 11550 4100
 Connection ~ 10400 3050
 Wire Wire Line
@@
 Wire Wire Line
 	10200 3300 10950 3300
-Wire Wire Line
-	11450 3050 12150 3050
-Wire Wire Line
-	12150 3050 12150 4550
 Wire Notes Line
 	9250 4850 9250 5900
@@
 Wire Wire Line
 	7350 6400 7350 8200
-Wire Wire Line
-	10850 3800 10850 4100
 Wire Wire Line
 	11050 1800 11050 1650
@@
 	2400 7050 3300 7050
 Wire Wire Line
-	2900 1150 2900 1100
-Wire Wire Line
-	2900 1100 4500 1100
-Wire Wire Line
-	4500 1100 4500 1150
-Connection ~ 3700 1100
-Wire Wire Line
 	3700 3600 3700 3550
 Wire Wire Line
@@
 Connection ~ 7600 1100
 Connection ~ 8050 1100
-Wire Wire Line
-	14900 5400 14400 5400
-Wire Wire Line
-	14400 5400 14400 5300
-Wire Wire Line
-	15400 5400 15800 5400
-Wire Wire Line
-	15800 5400 15800 5700
-Wire Wire Line
-	10200 3900 10200 4100
-Wire Wire Line
-	15150 5350 15150 5100
 Wire Wire Line
 	8600 9400 8600 9500
@@
 Text Notes 8450 5850 2    60   ~ 0
 ISP for AVR (Optional)
-Text Label 15150 5100 1    60   ~ 0
-PD7
-Text Label 10200 4100 3    60   ~ 0
-PD7
 Wire Wire Line
 	15350 3400 15350 3700
@@
 Wire Wire Line
 	15050 3650 15050 3800
-Text Notes 2650 4000 0    60   ~ 0
+Text Notes 3950 1750 0    60   ~ 0
 Main Processor
 Text Notes 8650 4250 0    60   ~ 0
@@
 SPI-SCK
 NoConn ~ 1800 2550
+$Comp
+L ROTARY-ENCODER S?
+U 1 1 58EE7837
+P 15250 4500
+F 0 "S?" H 15600 4500 60  0000 C CNN
+F 1 "ROTARY-ENCODER" H 15300 4850 60  0000 C CNN
+F 2 "" H 15250 4500 60  0001 C CNN
+F 3 "" H 15250 4500 60  0001 C CNN
+	1    15250 4500
+	0    1    1    0
+$EndComp
+Wire Wire Line
+	10200 3400 10950 3400
+Text Label 10550 3400 0    60   ~ 0
+PD2
+Wire Wire Line
+	10200 3600 10900 3600
+Text Label 10500 3600 0    60   ~ 0
+PD4
+Wire Wire Line
+	14800 4300 14400 4300
+Text Label 14400 4300 0    60   ~ 0
+PD2
+Wire Wire Line
+	14800 4700 14400 4700
+Text Label 14400 4700 0    60   ~ 0
+PD4
+Wire Wire Line
+	14800 4500 14150 4500
+Wire Wire Line
+	14150 4500 14150 4850
+NoConn ~ 10200 3800
+NoConn ~ 10200 3900
+Text Notes 5450 1500 0    60   ~ 0
+ESP8266 Board has 12K pullups \non GPIO0 and CHIP-EN
+NoConn ~ 3000 2700
 $EndSCHEMATC
