File: hardware/kicad/InternetRadioMinibox/InternetRadioMiniBox.sch (KiCad schematic (older format))
At the start: 56 parts, among them IC2 ATMEGA328P-P, IC3 23K256, IC4 VS1011e, IC5 LM386, M1 TSR1-2450, M2 TSR1-2433, M3 TSR1-2433, P1 CONN_01X02, P2 CONN_01X02, P3 CONN_01X02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

Commit message: Removed the SRAM component from the schematic.
Parts:
- removed C20: 22u, Capacitors_ThroughHole:CP_Radial_D5.0mm_P2.00mm, symbol CP
- removed C21: 100n, Capacitors_SMD:C_0805_HandSoldering, symbol C
- removed IC3: 23K256, Housings_SOIC:SOIC-8_3.9x4.9mm_Pitch1.27mm, symbol 23K256
- removed R10, R9: 10K, Resistors_SMD:R_0805_HandSoldering, symbol R
Connections:
- net labels removed: SPI-RAM-CS
- wire segments 220 -> 237
- no-connect marks 28 -> 27
Other:
- note removed: "RING \nBUFFER"

Commit message: Added back the SPI RAM 23K256 as still required for buffering
Parts:
- added C?: 100n, symbol C
- added C?: 22u, Capacitors_ThroughHole:CP_Radial_D5.0mm_P2.00mm, symbol CP
- added IC?: 23K256, DIL, symbol 23K256
- added R? (x2): 10K, symbol R
Connections:
- net labels added: SPI-RAM-CS
- wire segments 237 -> 216
- no-connect marks 27 -> 28

Commit message: Now using the Adafruit MusicMaker with Amp
Parts:
- removed C10, C11: 1u-100u, symbol CP
- removed C12: 220u, maker:C_RADIAL_D8_P3.5, symbol CP
- removed C13: 50n, Capacitors_SMD:C_0805_HandSoldering, symbol C
- removed C16, C18: 22u, Capacitors_ThroughHole:CP_Radial_D5.0mm_P2.00mm, symbol CP
- removed C17, C19, C9: 100n, Capacitors_SMD:C_0805_HandSoldering, symbol C
- removed C7, C8: 33p, Capacitors_SMD:C_0805_HandSoldering, symbol C
- removed IC4: VS1011e, Housings_SOIC:SOIC-28W_7.5x17.9mm_Pitch1.27mm, symbol VS1011e
- removed IC5: LM386, Housings_SOIC:SOIC-8-1EP_3.9x4.9mm_Pitch1.27mm, symbol LM386-RESCUE-InternetRadioMiniBox
- removed P8: CONN_ALT_AMP, Connect:PINHEAD1-2, symbol CONN_01X02
- removed R11: 10M, Resistors_SMD:R_0805_HandSoldering, symbol R
- removed R12: 100k, Resistors_SMD:R_0805_HandSoldering, symbol R
- removed R13, R14, R15, R16: 100K, Resistors_SMD:R_0805_HandSoldering, symbol R
- removed R17, R18: 4.7K, Resistors_SMD:R_0805_HandSoldering, symbol R
- removed R19: 47K, Resistors_SMD:R_0805_HandSoldering, symbol R
- removed R20: 10, Resistors_SMD:R_0805_HandSoldering, symbol R
- removed Y2: 12.288 MHz, symbol Crystal
- added SOM?: Adafruit-Feather-MusicMaker/Amp, symbol Adafruit-Feather-MusicMaker/Amp
Connections:
- net labels removed: AUDIO-LEFT, AUDIO-RIGHT, SPEAKER+
- wire segments 216 -> 162
- no-connect marks 28 -> 26
Other:
- note added: "BUffer"
- note added: "Pinouts Feather MusicMaker/Amp"
- note added: "SPI used internally \nfor WIFI"
- note added: "TO DO:\n - Power supplies"
- note removed: "AMP"
- note removed: "Depending on \nload resistance"
- note removed: "MP3\nDECODER"
- moved on the sheet: C1, C2, C3, C4, C5, C6, C?, D1, D2, IC2, IC?, M2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
